File: hardware/LED_Board/LEDBoard_template/LEDBoard_template.kicad_pcb (KiCad board)
At the start: 4 copper layers, 260 x 111.2 mm, 108 parts, among them J101 Conn_01x05, J102 NTC, J103 Conn_01x04, J104 Conn_01x04, J105 Conn_01x05, J106 FAN Connector, J201 NTC, Q101 BSS138, Q201 BSS138, U101 L6982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

Commit message: Working lamp pcb
Parts:
- added REF**: 3.45MM_NOTPLATED, Mounting_Holes:3.45MM_NOTPLATED, F.Cu at (117.0, 116.0)
- added REF**: 3.2mm_plated, Mounting_Holes:3.2mm_plated, F.Cu at (355.6, 110.3)
Other:
- board text added: "CC-BY-SA-NC"
- board text added: "F4IHX"
- board text added: "GreenLight Plant"
