File: hardware/LED_Board/LEDBoard_template/LEDBoard_template.kicad_sch (KiCad schematic)
At the start: 51 parts, among them J101 Conn_01x05, J102 NTC, J103 Conn_01x04, J104 Conn_01x04, J105 Conn_01x05, J106 FAN Connector, Q101 BSS138, U101 L6982, U102 22uH, U103 ADP8140ACPZ

Commit message: Working lamp pcb
Parts:
- R104: value 5k -> 3k
- R107: value 7.32k -> 15k
Other:
- note added: "Settings for about 150mA"
Changed lines of the file:
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@@
+    (effects (font (size 1.27 1.27)) (justify left bottom))
+  )
+  (text "Settings for about 150mA" (at 60.325 106.68 0)
     (effects (font (size 1.27 1.27)) (justify left bottom))
   )
@@
       (effects (font (size 0.635 0.635)))
     )
-    (property "Value" "5k" (id 1) (at 59.69 85.09 0)
+    (property "Value" "3k" (id 1) (at 59.69 85.09 0)
       (effects (font (size 0.635 0.635)))
     )
@@
       (effects (font (size 0.635 0.635)))
     )
-    (property "Value" "7.32k" (id 1) (at 83.82 90.805 0)
+    (property "Value" "15k" (id 1) (at 83.82 90.805 0)
       (effects (font (size 0.635 0.635)))
     )
@@
     )
     (path "/7255b086-c0cd-4fbd-a16b-411b9c6522b1"
-      (reference "R104") (unit 1) (value "5k") (footprint "SM0603")
+      (reference "R104") (unit 1) (value "3k") (footprint "SM0603")
     )
     (path "/e1feab75-c24f-4da2-91f6-19bdc7977cf2"
@@
     )
     (path "/f948e784-6f7a-45b9-8898-a8c09ac06842"
-      (reference "R107") (unit 1) (value "7.32k") (footprint "SM0603")
+      (reference "R107") (unit 1) (value "15k") (footprint "SM0603")
     )
     (path "/c24150c6-b6e6-4a0f-b908-d8d5e70f02ef"
@@
     )
     (path "/f1dd9b7f-4356-4e84-bf2c-fb8cc5eb7ed1/68f8542a-34f4-484a-8cfe-ce4490bb021d"
-      (reference "R204") (unit 1) (value "5k") (footprint "SM0603")
+      (reference "R204") (unit 1) (value "3k") (footprint "SM0603")
     )
     (path "/f1dd9b7f-4356-4e84-bf2c-fb8cc5eb7ed1/49775adc-3d93-4fea-ac27-d4d05a56a2e7"
@@
     )
     (path "/f1dd9b7f-4356-4e84-bf2c-fb8cc5eb7ed1/3c3c4e3c-a35b-4270-b84a-f9a5a649cd34"
-      (reference "R207") (unit 1) (value "7.32k") (footprint "SM0603")
+      (reference "R207") (unit 1) (value "15k") (footprint "SM0603")
     )
     (path "/f1dd9b7f-4356-4e84-bf2c-fb8cc5eb7ed1/fac35319-4246-4b13-a029-eba8adc5638a"
