File: hardware/LED_Board/LEDBoard_template/led_stack.kicad_sch (KiCad schematic)
At the start: 46 parts, among them J201 NTC, Q201 BSS138, U201 L6982, U202 22uH, U203 ADP8140ACPZ

Commit message: Working lamp pcb
Parts:
- R204: value 5k -> 3k
- R207: value 7.32k -> 15k
Other:
- note added: "Settings for about 150mA"
Changed lines of the file:
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@@
+    (effects (font (size 1.27 1.27)) (justify left bottom))
+  )
+  (text "Settings for about 150mA" (at 111.125 133.35 0)
     (effects (font (size 1.27 1.27)) (justify left bottom))
   )
@@
       (effects (font (size 0.635 0.635)))
     )
-    (property "Value" "7.32k" (id 1) (at 140.97 118.745 0)
+    (property "Value" "15k" (id 1) (at 140.97 118.745 0)
       (effects (font (size 0.635 0.635)))
     )
@@
       (effects (font (size 0.635 0.635)))
     )
-    (property "Value" "5k" (id 1) (at 116.84 113.03 0)
-      (effects (font (size 0.635 0.635)))
-    )
+    (property "Value" "3k" (id 1) (at 116.84 113.03 0)
+      (effects (font (size 0.635 0.635)))
+    )
